File: BreakoutBodger Deluxe/Kicad/Atmega_328_breakout.kicad_pcb (KiCad board)
At the start: 2 copper layers, 73.8 x 62 mm, 83 parts, among them J1 Power_connector, J10 Device_Connector, J11 Power terminal, J12 Jack-DC, J13 1x2, J14 1x2, J15 1x2, J16 1x2, J17 Conn_01x06, J18 1x2, J19 1x2, J2 ADC_Connector, J20 1x2, J21 1x2, J22 1x2, J23 1x2, J24 1x2, J25 1x2, J26 1x2, J27 1x2, J28 1x2, J29 1x2, J3 Com_header, J30 Pin out, J4 PORB++_connector, J5 PORD_connector, J6 USB, J7 Conn_01x01, Q1 PMOS, SW1 SW_Push, SW2 SW_Push, U1 MCP1700-33, U2 TL071, U3 ATMEGA328P-AU, U4 L7805, U5 MCP2221, U6 NCP1117-5, Y1 Crystal

Commit message: Picture and increase in trace size
Routing:
- net /PC0: track 21.3 -> 22.7 mm
- net /PC3: track 24.8 -> 26.0 mm
- net /PC5(SCL): track 67.8 -> 68.9 mm
- net /PC4(SDA): track 71.4 -> 72.6 mm
- net /PC2: track 22.4 -> 23.6 mm
- net /PC1: track 20.5 -> 21.7 mm
Changed lines of the file:
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@@
     (thickness 1.6)
     (drawings 28)
-    (tracks 902)
+    (tracks 909)
     (zones 0)
     (modules 83)
@@
   )
   (setup
-    (last_trace_width 0.25)
+    (last_trace_width 1)
     (user_trace_width 0.16)
     (user_trace_width 0.25)
@@
   (segment (start 108.65 59.4) (end 109 59.4) (width 0.35) (layer F.Cu) (net 13))
   (segment (start 52.07 90.725) (end 52.07 88.834) (width 0.25) (layer F.Cu) (net 14))
+  (segment (start 89.281 113.157) (end 89.281 110.347) (width 1) (layer F.Cu) (net 15))
+  (segment (start 89.281 110.347) (end 90.024 109.604) (width 1) (layer F.Cu) (net 15))
+  (segment (start 90.024 109.604) (end 90.024 109.824) (width 1) (layer F.Cu) (net 15))
   (segment (start 89.972 109.53) (end 89.972 109.022) (width 0.35) (layer F.Cu) (net 15))
   (segment (start 89.972 109.022) (end 91.899956 107.094044) (width 0.35) (layer F.Cu) (net 15))
@@
   (segment (start 91.924932 99.007932) (end 88.487 95.57) (width 0.35) (layer F.Cu) (net 15))
   (segment (start 88.487 95.57) (end 88.487 94.42) (width 0.35) (layer F.Cu) (net 15))
-  (segment (start 89.281 113.157) (end 89.281 110.49) (width 0.25) (layer B.Cu) (net 15))
   (segment (start 89.281 110.49) (end 90.17 109.601) (width 0.25) (layer B.Cu) (net 15))
+  (segment (start 91.821 113.157) (end 91.821 110.347) (width 1) (layer F.Cu) (net 16))
+  (segment (start 91.821 110.347) (end 92.564 109.604) (width 1) (layer F.Cu) (net 16))
   (segment (start 92.650011 102.626827) (end 92.449967 102.826871) (width 0.35) (layer F.Cu) (net 16))
   (segment (start 92.474943 99.49711) (end 92.650011 99.672178) (width 0.35) (layer F.Cu) (net 16))
@@
   (segment (start 92.449967 107.847967) (end 92.512 107.91) (width 0.35) (layer F.Cu) (net 16))
   (segment (start 89.287 94.42) (end 89.287 95.57) (width 0.35) (layer F.Cu) (net 16))
-  (segment (start 91.821 113.157) (end 91.821 110.49) (width 0.25) (layer B.Cu) (net 16))
   (segment (start 91.821 110.49) (end 92.71 109.601) (width 0.25) (layer B.Cu) (net 16))
+  (segment (start 94.361 113.157) (end 94.361 110.347) (width 1) (layer F.Cu) (net 17))
+  (segment (start 94.361 110.347) (end 95.104 109.604) (width 1) (layer F.Cu) (net 17))
   (segment (start 95.052 109.022) (end 92.999978 106.969978) (width 0.35) (layer F.Cu) (net 17))
   (segment (start 93.200022 102.854649) (end 93.200022 99.410358) (width 0.35) (layer F.Cu) (net 17))
@@
   (segment (start 93.024954 95.882954) (end 90.737 93.595) (width 0.35) (layer F.Cu) (net 17))
   (segment (start 93.024954 99.23529) (end 93.024954 95.882954) (width 0.35) (layer F.Cu) (net 17))
-  (segment (start 94.361 113.157) (end 94.361 110.49) (width 0.25) (layer B.Cu) (net 17))
   (segment (start 94.361 110.49) (end 95.25 109.601) (width 0.25) (layer B.Cu) (net 17))
+  (segment (start 96.901 113.157) (end 96.901 110.347) (width 1) (layer F.Cu) (net 18))
+  (segment (start 96.901 110.347) (end 97.644 109.604) (width 1) (layer F.Cu) (net 18))
   (segment (start 97.592 109.022) (end 97.592 109.53) (width 0.35) (layer F.Cu) (net 18))
   (segment (start 93.574965 99.007468) (end 93.750033 99.182536) (width 0.35) (layer F.Cu) (net 18))
@@
   (segment (start 91.887 92.17) (end 93.574965 93.857965) (width 0.35) (layer F.Cu) (net 18))
   (segment (start 93.574965 93.857965) (end 93.574965 99.007468) (width 0.35) (layer F.Cu) (net 18))
-  (segment (start 96.901 113.157) (end 96.901 110.49) (width 0.25) (layer B.Cu) (net 18))
   (segment (start 96.901 110.49) (end 97.79 109.601) (width 0.25) (layer B.Cu) (net 18))
+  (segment (start 99.441 113.157) (end 99.441 110.347) (width 1) (layer F.Cu) (net 19))
+  (segment (start 99.441 110.347) (end 100.184 109.604) (width 1) (layer F.Cu) (net 19))
   (segment (start 63.88 69.5) (end 62.704999 70.675001) (width 0.25) (layer F.Cu) (net 19))
   (segment (start 62.704999 70.675001) (end 62.704999 72.742001) (width 0.25) (layer F.Cu) (net 19))
@@
   (segment (start 74.848 91.426) (end 70.6 87.178) (width 0.25) (layer F.Cu) (net 19))
   (via (at 74.848 91.426) (size 0.5) (drill 0.4) (layers F.Cu B.Cu) (net 19))
-  (segment (start 99.441 113.157) (end 99.441 110.49) (width 0.25) (layer B.Cu) (net 19))
   (segment (start 99.441 110.49) (end 100.33 109.601) (width 0.25) (layer B.Cu) (net 19))
+  (segment (start 101.981 113.157) (end 101.981 110.347) (width 1) (layer F.Cu) (net 20))
+  (segment (start 101.981 110.347) (end 102.724 109.604) (width 1) (layer F.Cu) (net 20))
   (segment (start 91.887 90.57) (end 94.674987 93.357987) (width 0.35) (layer F.Cu) (net 20))
   (segment (start 94.674987 98.551824) (end 94.850055 98.726892) (width 0.35) (layer F.Cu) (net 20))
@@
   (segment (start 64.517999 72.815999) (end 63.668 71.966) (width 0.25) (layer F.Cu) (net 20))
   (via (at 75.348 90.526) (size 0.5) (drill 0.4) (layers F.Cu B.Cu) (net 20))
-  (segment (start 101.981 113.157) (end 101.981 110.49) (width 0.25) (layer B.Cu) (net 20))
   (segment (start 101.981 110.49) (end 102.87 109.601) (width 0.25) (layer B.Cu) (net 20))
   (segment (start 85.38199 93.17501) (end 85.583997 93.17501) (width 0.35) (layer F.Cu) (net 21))
